Commit message: Deployment Latest

File: src/description/ros2_control.xacro (robot description, xacro)
@@ -1,26 +1,26 @@
 <?xml version="1.0"?>
 <robot xmlns:xacro="http://www.ros.org/wiki/xacro">
-    <ros2_control name="DiffDriveHardware" type="system">
-        <hardware>
-            <plugin>diffdrive_rpi/DiffDriveRpiHardware</plugin>
-            <param name="left_pwm_pin">12</param>
-            <param name="left_dir_pin">16</param>
-            <param name="right_pwm_pin">13</param>
-            <param name="right_dir_pin">26</param>
-            <param name="pwm_freq">20000</param>
-            <param name="wheel_radius">0.05</param>
-            <param name="wheel_separation">0.25</param>
-            <param name="max_wheel_speed">1.0</param>
-        </hardware>
-        <joint name="left_wheel_joint">
-            <command_interface name="velocity"/>
-            <state_interface name="position"/>
-            <state_interface name="velocity"/>
-        </joint>
-        <joint name="right_wheel_joint">
-            <command_interface name="velocity"/>
-            <state_interface name="position"/>
-            <state_interface name="velocity"/>
-        </joint>
-    </ros2_control>
+  <ros2_control name="DiffDriveHardware" type="system">
+    <hardware>
+      <plugin>fake_components/GenericSystem</plugin>
+      <param name="fake_sensor_commands">false</param>
+      <param name="state_following_offset">0.0</param>
+    </hardware>
+    <joint name="left_wheel_joint">
+      <command_interface name="velocity">
+        <param name="min">-10</param>
+        <param name="max">10</param>
+      </command_interface>
+      <state_interface name="position"/>
+      <state_interface name="velocity"/>
+    </joint>
+    <joint name="right_wheel_joint">
+      <command_interface name="velocity">
+        <param name="min">-10</param>
+        <param name="max">10</param>
+      </command_interface>
+      <state_interface name="position"/>
+      <state_interface name="velocity"/>
+    </joint>
+  </ros2_control>
 </robot>
