Commit message: Hardware Interface Update Arduino

File: src/description/lidar.xacro (robot description, xacro)
@@ -1,27 +1,31 @@
 <?xml version="1.0"?>
 <robot xmlns:xacro="http://www.ros.org/wiki/xacro" >
-<link name="lidar_link">
-  <inertial>
-    <origin xyz="0 0 0" rpy="0 0 0"/>
-    <mass value="0.125"/>
-    <inertia ixx="0.001"  ixy="0"  ixz="0" iyy="0.001" iyz="0" izz="0.001" />
-  </inertial>
-  <collision>
-    <origin xyz="0 0 0" rpy="0 0 0"/>
-    <geometry>
-       <cylinder radius="0.0508" length="0.055"/>
-    </geometry>
-  </collision>
-  <visual>
-    <origin xyz="0 0 0" rpy="0 0 0"/>
-    <geometry>
-       <cylinder radius="0.0508" length="0.055"/>
-    </geometry>
-  </visual>
-</link>
-<joint name="lidar_joint" type="fixed">
-  <parent link="chassis"/>
-  <child link="lidar_link"/>
-  <origin xyz="0.1 0 0.19" rpy="0 0 0"/>
-</joint>
+    <joint name="laser_joint" type="fixed">
+        <parent link="chassis"/>
+        <child link="laser_frame"/>
+        <origin xyz="0.122 0 0.212" rpy="0 0 0"/>
+    </joint>
+    <link name="laser_frame">
+        <visual>
+            <geometry>
+                <cylinder radius="0.05" length="0.04"/>
+            </geometry>
+            <material name="black"/>
+        </visual>
+        <visual>
+            <origin xyz="0 0 -0.05"/>
+            <geometry>
+                <cylinder radius="0.01" length="0.1"/>
+            </geometry>
+            <material name="black"/>
+        </visual>
+        <collision>
+            <geometry>
+                <cylinder radius="0.05" length="0.04"/>
+            </geometry>
+        </collision>
+        <xacro:inertial_cylinder mass="0.1" length="0.04" radius="0.05">
+            <origin xyz="0 0 0" rpy="0 0 0"/>
+        </xacro:inertial_cylinder>
+    </link>
 </robot>

File: src/description/ros2_control.xacro (robot description, xacro)
@@ -3,8 +3,17 @@
   <ros2_control name="DiffDriveHardware" type="system">
     <hardware>
-      <plugin>fake_components/GenericSystem</plugin>
-      <param name="fake_sensor_commands">false</param>
-      <param name="state_following_offset">0.0</param>
-    </hardware>
+        <plugin>diffdrive_arduino/DiffDriveArduinoHardware</plugin>
+        <param name="left_wheel_name">left_wheel_joint</param>
+        <param name="right_wheel_name">right_wheel_joint</param>
+        <param name="loop_rate">30</param>
+        <param name="device">/dev/serial/by-path/platform-fd500000.pcie-pci-0000:01:00.0-usb-0:1.3:1.0-port0</param>
+        <param name="baud_rate">57600</param>
+        <param name="timeout_ms">1000</param>
+        <param name="enc_counts_per_rev">3436</param>
+        <param name="pid_p">20</param>
+        <param name="pid_d">12</param>
+        <param name="pid_i">0</param>
+        <param name="pid_o">50</param>
+      </hardware>
     <joint name="left_wheel_joint">
       <command_interface name="velocity">
